Commit message: Add Robotiq 2F-85 + D405 end effector for mobile FR3 duo
- New end_effectors/robotiq_2f85_d405/ with:
    robotiq_2f85_d405.urdf.xacro        — attachment macro
    robotiq_2f85_d405_kinematics.urdf.xacro — links/joints/mimic (placeholder;
      replace with output of extract_gripper_urdf.py after running in Isaac Sim)
- franka_robot.xacro: add robotiq_2f85_d405 branch alongside franka_hand
- mobile_fr3_duo_v0_2.urdf.xacro: change default ee_id to robotiq_2f85_d405

Co-Authored-By: Claude Sonnet 4.6 <noreply@anthropic.com>

File: robots/common/franka_robot.xacro (robot description, xacro)
@@ -68,5 +68,19 @@
       />
     </xacro:if>
-    <xacro:if value="${hand and ee_id != 'none' and ee_id != 'franka_hand'}">
+    <!-- Robotiq 2F-85 + Intel RealSense D405 wrist camera -->
+    <xacro:if value="${hand and ee_id == 'robotiq_2f85_d405'}">
+      <xacro:include filename="$(find franka_description)/end_effectors/robotiq_2f85_d405/robotiq_2f85_d405.urdf.xacro"/>
+      <xacro:property name="connection"
+        value="${special_connection if special_connection != '' else robot_type + '_link8'}"/>
+      <xacro:robotiq_2f85_d405
+        connected_to="${arm_prefix}${connection}"
+        arm_prefix="${arm_prefix}"
+        robot_type="${robot_type}"
+        xyz_ee="${xyz_ee}"
+        rpy_ee="${rpy_ee}"
+        description_pkg="${description_pkg}"
+      />
+    </xacro:if>
+    <xacro:if value="${hand and ee_id != 'none' and ee_id != 'franka_hand' and ee_id != 'robotiq_2f85_d405'}">
       <xacro:include filename="$(find franka_description)/end_effectors/common/ee_with_one_link.xacro"/>
       <xacro:include filename="$(find franka_description)/end_effectors/common/utils.xacro"/>

File: robots/mobile_fr3_duo_v0_2/mobile_fr3_duo_v0_2.urdf.xacro (robot description, xacro)
@@ -11,5 +11,5 @@
   <xacro:arg name="hand" default="true"/>
   <!-- Which end-effector would be mounted at the flange?" -->
-  <xacro:arg name="ee_id" default="franka_hand"/>
+  <xacro:arg name="ee_id" default="robotiq_2f85_d405"/>
   <!-- Where is the end-effector connected to, if different from the robot flange?  -->
   <xacro:arg name="special_connection" default=""/>
