Commit message: Replace kinematics placeholder with USD-extracted values; fix flange rotation
- robotiq_2f85_d405_kinematics.urdf.xacro: replaced placeholder with real
  transforms extracted from FR3_robotiq_2f85.usd via extract_gripper_urdf.py
  (23 links, 22 joints, non-zero origins, mimic joints coupled to gripper_ctrl)
- robotiq_2f85_d405.urdf.xacro: set rpy_ee default to 0 0 -0.7853982 (-π/4)
  to match fr3v2_link8/fr3v2_ur_to_robotiq_joint rotation in USD

Co-Authored-By: Claude Sonnet 4.6 <noreply@anthropic.com>

File: end_effectors/robotiq_2f85_d405/robotiq_2f85_d405.urdf.xacro (robot description, xacro)
@@ -26,11 +26,10 @@
             robot_type:='fr3v2_1'
             xyz_ee:='0 0 0'
-            rpy_ee:='0 0 0'
+            rpy_ee:='0 0 -0.7853982'
             description_pkg:='franka_description'">
     <!--
-      Attachment joint: arm flange (link8) → ur_to_robotiq_link.
-      The xyz/rpy values should come from the USD joint
-      fr3v2_link8/fr3v2_ur_to_robotiq_joint — pass them via xyz_ee/rpy_ee
-      or leave at 0 0 0 if the USD joint has zero offset.
+      Attachment joint: arm flange (link8) → fr3v2_ur_to_robotiq_link.
+      rpy_ee default -π/4 comes from the fr3v2_link8/fr3v2_ur_to_robotiq_joint
+      in the USD — the UR coupling is rotated −45° about Z relative to the flange.
     -->
     <joint name="${arm_prefix}${robot_type}_ur_to_robotiq_joint" type="fixed">

File: end_effectors/robotiq_2f85_d405/robotiq_2f85_d405_kinematics.urdf.xacro (robot description, xacro)
@@ -3,175 +3,187 @@
   AUTO-GENERATED by franka_isaacSim/scripts/tooling/extract_gripper_urdf.py
   Source: assets/embodiments/fr3/FR3_robotiq_2f85.usd
-  THIS IS A PLACEHOLDER.  Run the extraction script inside Isaac Sim to
-  populate this file with actual kinematic data from the USD:
-      docker exec isaac-sim bash -c "
-        LD_LIBRARY_PATH=/isaac-sim/extscache/omni.usd.libs-1.0.1+69cbf6ad.lx64.r.cp311/bin \
-        /isaac-sim/python.sh /workspace/scripts/tooling/extract_gripper_urdf.py"
-  Then copy the output to this file:
-      cp /workspace/assets/embodiments/fr3/robotiq_2f85_d405_kinematics.urdf.xacro \
-         franka_description/end_effectors/robotiq_2f85_d405/robotiq_2f85_d405_kinematics.urdf.xacro
-  DO NOT EDIT this file by hand — regenerate from USD whenever kinematics change.
+  DO NOT EDIT by hand — regenerate from USD if kinematics change.
 -->
 <robot xmlns:xacro="http://www.ros.org/wiki/xacro">
+  <!--
+    Macro: robotiq_2f85_d405_kinematics
+    Params:
+      arm_prefix  — e.g. 'left_' or 'right_' for dual-arm setups ('' for single)
+  -->
   <xacro:macro name="robotiq_2f85_d405_kinematics" params="arm_prefix:=''">
-    <!-- ── Links ──────────────────────────────────────────────────────────── -->
-    <link name="${arm_prefix}fr3v2_ur_to_robotiq_link"/>
-    <link name="${arm_prefix}fr3v2_robotiq_85_base_adapter_link"/>
-    <link name="${arm_prefix}fr3v2_robotiq_85_base_link"/>
-    <link name="${arm_prefix}fr3v2_robotiq_85_left_knuckle_link"/>
-    <link name="${arm_prefix}fr3v2_robotiq_85_right_knuckle_link"/>
-    <link name="${arm_prefix}fr3v2_robotiq_85_left_inner_knuckle_link"/>
-    <link name="${arm_prefix}fr3v2_robotiq_85_right_inner_knuckle_link"/>
-    <link name="${arm_prefix}fr3v2_robotiq_85_left_finger_link"/>
-    <link name="${arm_prefix}fr3v2_robotiq_85_right_finger_link"/>
-    <link name="${arm_prefix}fr3v2_robotiq_85_left_finger_tip_link"/>
-    <link name="${arm_prefix}fr3v2_robotiq_85_right_finger_tip_link"/>
-    <link name="${arm_prefix}fr3v2_tcp"/>
-    <link name="${arm_prefix}fr3v2_wrist_cam_mount_link"/>
-    <link name="${arm_prefix}fr3v2_d405_camera_link"/>
-    <link name="${arm_prefix}fr3v2_d405_color_frame"/>
-    <link name="${arm_prefix}fr3v2_d405_depth_frame"/>
-    <link name="${arm_prefix}fr3v2_d405_imu_link"/>
-    <link name="${arm_prefix}fr3v2_d405_infra1_frame"/>
-    <link name="${arm_prefix}fr3v2_d405_infra2_frame"/>
-    <link name="${arm_prefix}fr3v2_d405_color_optical_frame"/>
-    <link name="${arm_prefix}fr3v2_d405_depth_optical_frame"/>
-    <link name="${arm_prefix}fr3v2_d405_infra1_optical_frame"/>
-    <link name="${arm_prefix}fr3v2_d405_infra2_optical_frame"/>
-    <!-- ── Fixed joints (placeholder origins — replace with extracted values) -->
-    <joint name="${arm_prefix}fr3v2_gripper_side_joint" type="fixed">
+    <!-- ── Links ─────────────────────────────────────────── -->
+    <link name="${arm_prefix}d405_camera_link">
+    </link>
+    <link name="${arm_prefix}d405_color_frame">
+    </link>
+    <link name="${arm_prefix}d405_color_optical_frame">
+    </link>
+    <link name="${arm_prefix}d405_depth_frame">
+    </link>
+    <link name="${arm_prefix}d405_depth_optical_frame">
+    </link>
+    <link name="${arm_prefix}d405_imu_link">
+    </link>
+    <link name="${arm_prefix}d405_infra1_frame">
+    </link>
+    <link name="${arm_prefix}d405_infra1_optical_frame">
+    </link>
+    <link name="${arm_prefix}d405_infra2_frame">
+    </link>
+    <link name="${arm_prefix}d405_infra2_optical_frame">
+    </link>
+    <link name="${arm_prefix}robotiq_85_base_adapter_link">
+    </link>
+    <link name="${arm_prefix}robotiq_85_base_link">
+    </link>
+    <link name="${arm_prefix}robotiq_85_left_finger_link">
+    </link>
+    <link name="${arm_prefix}robotiq_85_left_finger_tip_link">
+    </link>
+    <link name="${arm_prefix}robotiq_85_left_inner_knuckle_link">
+    </link>
+    <link name="${arm_prefix}robotiq_85_left_knuckle_link">
+    </link>
+    <link name="${arm_prefix}robotiq_85_right_finger_link">
+    </link>
+    <link name="${arm_prefix}robotiq_85_right_finger_tip_link">
+    </link>
+    <link name="${arm_prefix}robotiq_85_right_inner_knuckle_link">
+    </link>
+    <link name="${arm_prefix}robotiq_85_right_knuckle_link">
+    </link>
+    <link name="${arm_prefix}tcp">
+    </link>
+    <link name="${arm_prefix}fr3v2_ur_to_robotiq_link">
+    </link>
+    <link name="${arm_prefix}wrist_cam_mount_link">
+    </link>
+    <!-- ── Joints ────────────────────────────────────────── -->
+    <joint name="${arm_prefix}d405_camera_joint" type="fixed">
+      <parent link="${arm_prefix}wrist_cam_mount_link"/>
+      <child  link="${arm_prefix}d405_camera_link"/>
+      <origin xyz="0.00000000 0.04100000 0.00810000" rpy="0.34904950 -0.00000000 0.00000000"/>
+    </joint>
+    <joint name="${arm_prefix}d405_color_joint" type="fixed">
+      <parent link="${arm_prefix}d405_camera_link"/>
+      <child  link="${arm_prefix}d405_color_frame"/>
+      <origin xyz="0.00000000 0.00000000 0.00000000" rpy="0.00000000 -0.00000000 0.00000000"/>
+    </joint>
+    <joint name="${arm_prefix}d405_color_optical_joint" type="fixed">
+      <parent link="${arm_prefix}d405_color_frame"/>
+      <child  link="${arm_prefix}d405_color_optical_frame"/>
+      <origin xyz="0.00000000 0.00000000 0.00000000" rpy="-1.57079633 -0.00000000 -1.57079633"/>
+    </joint>
+    <joint name="${arm_prefix}d405_depth_joint" type="fixed">
+      <parent link="${arm_prefix}d405_camera_link"/>
+      <child  link="${arm_prefix}d405_depth_frame"/>
+      <origin xyz="0.00000000 0.00000000 0.00000000" rpy="0.00000000 -0.00000000 0.00000000"/>
+    </joint>
+    <joint name="${arm_prefix}d405_depth_optical_joint" type="fixed">
+      <parent link="${arm_prefix}d405_depth_frame"/>
+      <child  link="${arm_prefix}d405_depth_optical_frame"/>
+      <origin xyz="0.00000000 0.00000000 0.00000000" rpy="-1.57079633 -0.00000000 -1.57079633"/>
+    </joint>
+    <joint name="${arm_prefix}d405_imu_joint" type="fixed">
+      <parent link="${arm_prefix}d405_camera_link"/>
+      <child  link="${arm_prefix}d405_imu_link"/>
+      <origin xyz="0.00000000 0.00000000 0.00000000" rpy="0.00000000 -0.00000000 0.00000000"/>
+    </joint>
+    <joint name="${arm_prefix}d405_infra1_joint" type="fixed">
+      <parent link="${arm_prefix}d405_camera_link"/>
+      <child  link="${arm_prefix}d405_infra1_frame"/>
+      <origin xyz="0.00000000 -0.01500000 0.00000000" rpy="0.00000000 -0.00000000 0.00000000"/>
+    </joint>
+    <joint name="${arm_prefix}d405_infra1_optical_joint" type="fixed">
+      <parent link="${arm_prefix}d405_infra1_frame"/>
+      <child  link="${arm_prefix}d405_infra1_optical_frame"/>
+      <origin xyz="0.00000000 0.00000000 0.00000000" rpy="-1.57079633 -0.00000000 -1.57079633"/>
+    </joint>
+    <joint name="${arm_prefix}d405_infra2_joint" type="fixed">
+      <parent link="${arm_prefix}d405_camera_link"/>
+      <child  link="${arm_prefix}d405_infra2_frame"/>
+      <origin xyz="0.00000000 0.01500000 0.00000000" rpy="0.00000000 -0.00000000 0.00000000"/>
+    </joint>
+    <joint name="${arm_prefix}d405_infra2_optical_joint" type="fixed">
+      <parent link="${arm_prefix}d405_infra2_frame"/>
+      <child  link="${arm_prefix}d405_infra2_optical_frame"/>
+      <origin xyz="0.00000000 0.00000000 0.00000000" rpy="-1.57079633 -0.00000000 -1.57079633"/>
+    </joint>
+    <joint name="${arm_prefix}gripper_ctrl" type="revolute">
+      <parent link="${arm_prefix}robotiq_85_base_link"/>
+      <child  link="${arm_prefix}robotiq_85_left_knuckle_link"/>
+      <origin xyz="0.03060100 0.00000000 0.05490500" rpy="0.00000000 -0.00000000 0.00000000"/>
+      <axis xyz="0 1 0"/>
+      <limit lower="0.00000000" upper="0.80000660" effort="200" velocity="0.5"/>
+    </joint>
+    <joint name="${arm_prefix}gripper_side_joint" type="fixed">
       <parent link="${arm_prefix}fr3v2_ur_to_robotiq_link"/>
-      <child  link="${arm_prefix}fr3v2_robotiq_85_base_adapter_link"/>
-      <origin xyz="0 0 0" rpy="0 0 0"/>
+      <child  link="${arm_prefix}robotiq_85_base_adapter_link"/>
+      <origin xyz="0.00000000 0.00000000 0.01100000" rpy="0.00000000 -0.00000000 0.00000000"/>
     </joint>
-    <joint name="${arm_prefix}fr3v2_robotiq_85_base_joint" type="fixed">
-      <parent link="${arm_prefix}fr3v2_robotiq_85_base_adapter_link"/>
-      <child  link="${arm_prefix}fr3v2_robotiq_85_base_link"/>
-      <origin xyz="0 0 0" rpy="0 0 0"/>
+    <joint name="${arm_prefix}robotiq_85_base_joint" type="fixed">
+      <parent link="${arm_prefix}robotiq_85_base_adapter_link"/>
+      <child  link="${arm_prefix}robotiq_85_base_link"/>
+      <origin xyz="0.00000000 0.00000000 0.00000000" rpy="0.00000000 -0.00000000 -0.78539820"/>
     </joint>
-    <joint name="${arm_prefix}fr3v2_tcp_joint" type="fixed">
-      <parent link="${arm_prefix}fr3v2_robotiq_85_base_link"/>
-      <child  link="${arm_prefix}fr3v2_tcp"/>
-      <origin xyz="0 0 0.1034" rpy="0 0 0"/>
+    <joint name="${arm_prefix}robotiq_85_left_finger_joint" type="fixed">
+      <parent link="${arm_prefix}robotiq_85_left_knuckle_link"/>
+      <child  link="${arm_prefix}robotiq_85_left_finger_link"/>
+      <origin xyz="0.03152600 0.00000000 -0.00376300" rpy="0.00000000 -0.00000000 0.00000000"/>
     </joint>
-    <joint name="${arm_prefix}fr3v2_wrist_cam_mount_joint" type="fixed">
-      <parent link="${arm_prefix}fr3v2_robotiq_85_base_link"/>
-      <child  link="${arm_prefix}fr3v2_wrist_cam_mount_link"/>
-      <origin xyz="0 0 0" rpy="0 0 0"/>
+    <joint name="${arm_prefix}robotiq_85_left_finger_tip_joint" type="revolute">
+      <parent link="${arm_prefix}robotiq_85_left_finger_link"/>
+      <child  link="${arm_prefix}robotiq_85_left_finger_tip_link"/>
+      <origin xyz="0.00563100 0.00000000 0.04718500" rpy="0.00000000 -0.00000000 0.00000000"/>
+      <axis xyz="0 1 0"/>
+      <limit lower="-17453292.51994330" upper="17453292.51994330" effort="200" velocity="0.5"/>
+      <mimic joint="${arm_prefix}gripper_ctrl" multiplier="-1.0000" offset="0.0000"/>
     </joint>
-    <!-- ── Gripper revolute joints ────────────────────────────────────────── -->
-    <!-- Single driven DOF; other fingers follow via <mimic> -->
-    <joint name="${arm_prefix}fr3v2_robotiq_85_left_knuckle_joint" type="revolute">
-      <parent link="${arm_prefix}fr3v2_robotiq_85_base_link"/>
-      <child  link="${arm_prefix}fr3v2_robotiq_85_left_knuckle_link"/>
-      <origin xyz="0 0 0" rpy="0 0 0"/>
+    <joint name="${arm_prefix}robotiq_85_left_inner_knuckle_joint" type="revolute">
+      <parent link="${arm_prefix}robotiq_85_base_link"/>
+      <child  link="${arm_prefix}robotiq_85_left_inner_knuckle_link"/>
+      <origin xyz="0.01270000 0.00000000 0.06142000" rpy="0.00000000 -0.00000000 0.00000000"/>
       <axis xyz="0 1 0"/>
-      <limit lower="0" upper="0.80286" effort="200" velocity="0.5"/>
+      <limit lower="-17453292.51994330" upper="17453292.51994330" effort="200" velocity="0.5"/>
+      <mimic joint="${arm_prefix}gripper_ctrl" multiplier="1.0000" offset="0.0000"/>
     </joint>
-    <joint name="${arm_prefix}fr3v2_robotiq_85_right_knuckle_joint" type="revolute">
-      <parent link="${arm_prefix}fr3v2_robotiq_85_base_link"/>
-      <child  link="${arm_prefix}fr3v2_robotiq_85_right_knuckle_link"/>
-      <origin xyz="0 0 0" rpy="0 0 0"/>
+    <joint name="${arm_prefix}robotiq_85_right_finger_joint" type="fixed">
+      <parent link="${arm_prefix}robotiq_85_right_knuckle_link"/>
+      <child  link="${arm_prefix}robotiq_85_right_finger_link"/>
+      <origin xyz="-0.03152600 0.00000000 -0.00376300" rpy="0.00000000 -0.00000000 0.00000000"/>
+    </joint>
+    <joint name="${arm_prefix}robotiq_85_right_finger_tip_joint" type="revolute">
+      <parent link="${arm_prefix}robotiq_85_right_finger_link"/>
+      <child  link="${arm_prefix}robotiq_85_right_finger_tip_link"/>
+      <origin xyz="-0.00563100 0.00000000 0.04718500" rpy="0.00000000 -0.00000000 0.00000000"/>
       <axis xyz="0 1 0"/>
-      <limit lower="0" upper="0.80286" effort="200" velocity="0.5"/>
-      <mimic joint="${arm_prefix}fr3v2_robotiq_85_left_knuckle_joint"
-             multiplier="1.0" offset="0.0"/>
+      <limit lower="-17453292.51994330" upper="17453292.51994330" effort="200" velocity="0.5"/>
+      <mimic joint="${arm_prefix}gripper_ctrl" multiplier="1.0000" offset="0.0000"/>
     </joint>
-    <joint name="${arm_prefix}fr3v2_robotiq_85_left_inner_knuckle_joint" type="revolute">
-      <parent link="${arm_prefix}fr3v2_robotiq_85_base_link"/>
-      <child  link="${arm_prefix}fr3v2_robotiq_85_left_inner_knuckle_link"/>
-      <origin xyz="0 0 0" rpy="0 0 0"/>
+    <joint name="${arm_prefix}robotiq_85_right_inner_knuckle_joint" type="revolute">
+      <parent link="${arm_prefix}robotiq_85_base_link"/>
+      <child  link="${arm_prefix}robotiq_85_right_inner_knuckle_link"/>
+      <origin xyz="-0.01270000 0.00000000 0.06142000" rpy="0.00000000 -0.00000000 0.00000000"/>
       <axis xyz="0 1 0"/>
-      <limit lower="0" upper="0.80286" effort="200" velocity="0.5"/>
-      <mimic joint="${arm_prefix}fr3v2_robotiq_85_left_knuckle_joint"
-             multiplier="1.0" offset="0.0"/>
+      <limit lower="-17453292.51994330" upper="17453292.51994330" effort="200" velocity="0.5"/>
+      <mimic joint="${arm_prefix}gripper_ctrl" multiplier="-1.0000" offset="0.0000"/>
     </joint>
-    <joint name="${arm_prefix}fr3v2_robotiq_85_right_inner_knuckle_joint" type="revolute">
-      <parent link="${arm_prefix}fr3v2_robotiq_85_base_link"/>
-      <child  link="${arm_prefix}fr3v2_robotiq_85_right_inner_knuckle_link"/>
-      <origin xyz="0 0 0" rpy="0 0 0"/>
+    <joint name="${arm_prefix}robotiq_85_right_knuckle_joint" type="revolute">
+      <parent link="${arm_prefix}robotiq_85_base_link"/>
+      <child  link="${arm_prefix}robotiq_85_right_knuckle_link"/>
+      <origin xyz="-0.03060100 0.00000000 0.05490500" rpy="0.00000000 -0.00000000 0.00000000"/>
       <axis xyz="0 1 0"/>
-      <limit lower="0" upper="0.80286" effort="200" velocity="0.5"/>
-      <mimic joint="${arm_prefix}fr3v2_robotiq_85_left_knuckle_joint"
-             multiplier="1.0" offset="0.0"/>
+      <limit lower="-0.80000660" upper="0.00000000" effort="200" velocity="0.5"/>
+      <mimic joint="${arm_prefix}gripper_ctrl" multiplier="-1.0000" offset="0.0000"/>
     </joint>
-    <joint name="${arm_prefix}fr3v2_robotiq_85_left_finger_tip_joint" type="revolute">
-      <parent link="${arm_prefix}fr3v2_robotiq_85_left_knuckle_link"/>
-      <child  link="${arm_prefix}fr3v2_robotiq_85_left_finger_tip_link"/>
-      <origin xyz="0 0 0" rpy="0 0 0"/>
-      <axis xyz="0 1 0"/>
-      <limit lower="-0.80286" upper="0" effort="200" velocity="0.5"/>
-      <mimic joint="${arm_prefix}fr3v2_robotiq_85_left_knuckle_joint"
-             multiplier="-1.0" offset="0.0"/>
+    <joint name="${arm_prefix}tcp_joint" type="fixed">
+      <parent link="${arm_prefix}robotiq_85_base_link"/>
+      <child  link="${arm_prefix}tcp"/>
+      <origin xyz="0.00000000 0.00000000 0.10340000" rpy="0.00000000 -0.00000000 0.00000000"/>
     </joint>
-    <joint name="${arm_prefix}fr3v2_robotiq_85_right_finger_tip_joint" type="revolute">
-      <parent link="${arm_prefix}fr3v2_robotiq_85_right_knuckle_link"/>
-      <child  link="${arm_prefix}fr3v2_robotiq_85_right_finger_tip_link"/>
-      <origin xyz="0 0 0" rpy="0 0 0"/>
-      <axis xyz="0 1 0"/>
-      <limit lower="-0.80286" upper="0" effort="200" velocity="0.5"/>
-      <mimic joint="${arm_prefix}fr3v2_robotiq_85_left_knuckle_joint"
-             multiplier="-1.0" offset="0.0"/>
-    </joint>
-    <joint name="${arm_prefix}fr3v2_robotiq_85_left_finger_joint" type="fixed">
-      <parent link="${arm_prefix}fr3v2_robotiq_85_left_inner_knuckle_link"/>
-      <child  link="${arm_prefix}fr3v2_robotiq_85_left_finger_link"/>
-      <origin xyz="0 0 0" rpy="0 0 0"/>
-    </joint>
-    <joint name="${arm_prefix}fr3v2_robotiq_85_right_finger_joint" type="fixed">
-      <parent link="${arm_prefix}fr3v2_robotiq_85_right_inner_knuckle_link"/>
-      <child  link="${arm_prefix}fr3v2_robotiq_85_right_finger_link"/>
-      <origin xyz="0 0 0" rpy="0 0 0"/>
-    </joint>
-    <!-- ── Camera chain ───────────────────────────────────────────────────── -->
-    <joint name="${arm_prefix}fr3v2_d405_camera_joint" type="fixed">
-      <parent link="${arm_prefix}fr3v2_wrist_cam_mount_link"/>
-      <child  link="${arm_prefix}fr3v2_d405_camera_link"/>
-      <origin xyz="0 0 0" rpy="0 0 0"/>
-    </joint>
-    <joint name="${arm_prefix}fr3v2_d405_color_joint" type="fixed">
-      <parent link="${arm_prefix}fr3v2_d405_camera_link"/>
-      <child  link="${arm_prefix}fr3v2_d405_color_frame"/>
-      <origin xyz="0 0 0" rpy="0 0 0"/>
-    </joint>
-    <joint name="${arm_prefix}fr3v2_d405_depth_joint" type="fixed">
-      <parent link="${arm_prefix}fr3v2_d405_camera_link"/>
-      <child  link="${arm_prefix}fr3v2_d405_depth_frame"/>
-      <origin xyz="0 0 0" rpy="0 0 0"/>
-    </joint>
-    <joint name="${arm_prefix}fr3v2_d405_imu_joint" type="fixed">
-      <parent link="${arm_prefix}fr3v2_d405_camera_link"/>
-      <child  link="${arm_prefix}fr3v2_d405_imu_link"/>
-      <origin xyz="0 0 0" rpy="0 0 0"/>
-    </joint>
-    <joint name="${arm_prefix}fr3v2_d405_infra1_joint" type="fixed">
-      <parent link="${arm_prefix}fr3v2_d405_camera_link"/>
-      <child  link="${arm_prefix}fr3v2_d405_infra1_frame"/>
-      <origin xyz="0 0 0" rpy="0 0 0"/>
-    </joint>
-    <joint name="${arm_prefix}fr3v2_d405_infra2_joint" type="fixed">
-      <parent link="${arm_prefix}fr3v2_d405_camera_link"/>
-      <child  link="${arm_prefix}fr3v2_d405_infra2_frame"/>
-      <origin xyz="0 0 0" rpy="0 0 0"/>
-    </joint>
-    <joint name="${arm_prefix}fr3v2_d405_color_optical_joint" type="fixed">
-      <parent link="${arm_prefix}fr3v2_d405_color_frame"/>
-      <child  link="${arm_prefix}fr3v2_d405_color_optical_frame"/>
-      <origin xyz="0 0 0" rpy="${-pi/2} 0 ${-pi/2}"/>
-    </joint>
-    <joint name="${arm_prefix}fr3v2_d405_depth_optical_joint" type="fixed">
-      <parent link="${arm_prefix}fr3v2_d405_depth_frame"/>
-      <child  link="${arm_prefix}fr3v2_d405_depth_optical_frame"/>
-      <origin xyz="0 0 0" rpy="${-pi/2} 0 ${-pi/2}"/>
-    </joint>
-    <joint name="${arm_prefix}fr3v2_d405_infra1_optical_joint" type="fixed">
-      <parent link="${arm_prefix}fr3v2_d405_infra1_frame"/>
-      <child  link="${arm_prefix}fr3v2_d405_infra1_optical_frame"/>
-      <origin xyz="0 0 0" rpy="${-pi/2} 0 ${-pi/2}"/>
-    </joint>
-    <joint name="${arm_prefix}fr3v2_d405_infra2_optical_joint" type="fixed">
-      <parent link="${arm_prefix}fr3v2_d405_infra2_frame"/>
-      <child  link="${arm_prefix}fr3v2_d405_infra2_optical_frame"/>
-      <origin xyz="0 0 0" rpy="${-pi/2} 0 ${-pi/2}"/>
+    <joint name="${arm_prefix}wrist_cam_mount_joint" type="fixed">
+      <parent link="${arm_prefix}robotiq_85_base_link"/>
+      <child  link="${arm_prefix}wrist_cam_mount_link"/>
+      <origin xyz="0.00000000 0.02700000 0.03630000" rpy="0.00000000 -0.00000000 0.00000000"/>
     </joint>
   </xacro:macro>
