Commit message: Add Robotiq 2F-85 + D405 gripper visual meshes and bundling script
- Add <visual> elements to robotiq_2f85_d405_kinematics.urdf.xacro for all
  12 gripper/camera links; add description_pkg param for mesh path resolution
- Add 12 STL mesh files extracted from FR3_robotiq_2f85.usd via pxr prototype
  traversal (arm adapter, base, knuckles, fingers, fingertips, wrist cam mount,
  D405 camera body)
- Add scripts/bundle_web_urdf.sh to zip URDF + all referenced meshes with
  relative paths for upload to web URDF viewers

Co-Authored-By: Claude Sonnet 4.6 <noreply@anthropic.com>

File: end_effectors/robotiq_2f85_d405/robotiq_2f85_d405.urdf.xacro (robot description, xacro)
@@ -39,5 +39,5 @@
     </joint>
     <!-- All gripper + camera links and joints (prefixed for dual-arm safety) -->
-    <xacro:robotiq_2f85_d405_kinematics arm_prefix="${arm_prefix}"/>
+    <xacro:robotiq_2f85_d405_kinematics arm_prefix="${arm_prefix}" description_pkg="${description_pkg}"/>
   </xacro:macro>
 </robot>

File: end_effectors/robotiq_2f85_d405/robotiq_2f85_d405_kinematics.urdf.xacro (robot description, xacro)
@@ -3,4 +3,5 @@
   AUTO-GENERATED by franka_isaacSim/scripts/tooling/extract_gripper_urdf.py
   Source: assets/embodiments/fr3/FR3_robotiq_2f85.usd
+  Meshes extracted by: franka_isaacSim/scripts/tooling/extract_gripper_meshes.py
   DO NOT EDIT by hand — regenerate from USD if kinematics change.
 -->
@@ -9,9 +10,108 @@
     Macro: robotiq_2f85_d405_kinematics
     Params:
-      arm_prefix  — e.g. 'left_' or 'right_' for dual-arm setups ('' for single)
+      arm_prefix      — e.g. 'left_' or 'right_' for dual-arm setups ('' for single)
+      description_pkg — ROS package containing meshes (default: franka_description)
   -->
-  <xacro:macro name="robotiq_2f85_d405_kinematics" params="arm_prefix:=''">
+  <xacro:macro name="robotiq_2f85_d405_kinematics"
+               params="arm_prefix:=''
+                       description_pkg:='franka_description'">
     <!-- ── Links ─────────────────────────────────────────── -->
+    <link name="${arm_prefix}fr3v2_ur_to_robotiq_link">
+      <visual>
+        <origin xyz="0 0 0" rpy="0 0 0"/>
+        <geometry>
+          <mesh filename="package://${description_pkg}/meshes/end_effectors/robotiq_2f85_d405/ur_to_robotiq_link.stl"/>
+        </geometry>
+      </visual>
+    </link>
+    <link name="${arm_prefix}robotiq_85_base_adapter_link">
+    </link>
+    <link name="${arm_prefix}robotiq_85_base_link">
+      <visual>
+        <origin xyz="0 0 0" rpy="0 0 0"/>
+        <geometry>
+          <mesh filename="package://${description_pkg}/meshes/end_effectors/robotiq_2f85_d405/robotiq_85_base_link.stl"/>
+        </geometry>
+      </visual>
+    </link>
+    <link name="${arm_prefix}robotiq_85_left_knuckle_link">
+      <visual>
+        <origin xyz="0 0 0" rpy="0 0 0"/>
+        <geometry>
+          <mesh filename="package://${description_pkg}/meshes/end_effectors/robotiq_2f85_d405/robotiq_85_left_knuckle_link.stl"/>
+        </geometry>
+      </visual>
+    </link>
+    <link name="${arm_prefix}robotiq_85_right_knuckle_link">
+      <visual>
+        <origin xyz="0 0 0" rpy="0 0 0"/>
+        <geometry>
+          <mesh filename="package://${description_pkg}/meshes/end_effectors/robotiq_2f85_d405/robotiq_85_right_knuckle_link.stl"/>
+        </geometry>
+      </visual>
+    </link>
+    <link name="${arm_prefix}robotiq_85_left_inner_knuckle_link">
+      <visual>
+        <origin xyz="0 0 0" rpy="0 0 0"/>
+        <geometry>
+          <mesh filename="package://${description_pkg}/meshes/end_effectors/robotiq_2f85_d405/robotiq_85_left_inner_knuckle_link.stl"/>
+        </geometry>
+      </visual>
+    </link>
+    <link name="${arm_prefix}robotiq_85_right_inner_knuckle_link">
+      <visual>
+        <origin xyz="0 0 0" rpy="0 0 0"/>
+        <geometry>
+          <mesh filename="package://${description_pkg}/meshes/end_effectors/robotiq_2f85_d405/robotiq_85_right_inner_knuckle_link.stl"/>
+        </geometry>
+      </visual>
+    </link>
+    <link name="${arm_prefix}robotiq_85_left_finger_link">
+      <visual>
+        <origin xyz="0 0 0" rpy="0 0 0"/>
+        <geometry>
+          <mesh filename="package://${description_pkg}/meshes/end_effectors/robotiq_2f85_d405/robotiq_85_left_finger_link.stl"/>
+        </geometry>
+      </visual>
+    </link>
+    <link name="${arm_prefix}robotiq_85_right_finger_link">
+      <visual>
+        <origin xyz="0 0 0" rpy="0 0 0"/>
+        <geometry>
+          <mesh filename="package://${description_pkg}/meshes/end_effectors/robotiq_2f85_d405/robotiq_85_right_finger_link.stl"/>
+        </geometry>
+      </visual>
+    </link>
+    <link name="${arm_prefix}robotiq_85_left_finger_tip_link">
+      <visual>
+        <origin xyz="0 0 0" rpy="0 0 0"/>
+        <geometry>
+          <mesh filename="package://${description_pkg}/meshes/end_effectors/robotiq_2f85_d405/robotiq_85_left_finger_tip_link.stl"/>
+        </geometry>
+      </visual>
+    </link>
+    <link name="${arm_prefix}robotiq_85_right_finger_tip_link">
+      <visual>
+        <origin xyz="0 0 0" rpy="0 0 0"/>
+        <geometry>
+          <mesh filename="package://${description_pkg}/meshes/end_effectors/robotiq_2f85_d405/robotiq_85_right_finger_tip_link.stl"/>
+        </geometry>
+      </visual>
+    </link>
+    <link name="${arm_prefix}wrist_cam_mount_link">
+      <visual>
+        <origin xyz="0 0 0" rpy="0 0 0"/>
+        <geometry>
+          <mesh filename="package://${description_pkg}/meshes/end_effectors/robotiq_2f85_d405/wrist_cam_mount_link.stl"/>
+        </geometry>
+      </visual>
+    </link>
     <link name="${arm_prefix}d405_camera_link">
+      <visual>
+        <origin xyz="0 0 0" rpy="0 0 0"/>
+        <geometry>
+          <mesh filename="package://${description_pkg}/meshes/end_effectors/robotiq_2f85_d405/d405_camera_link.stl"/>
+        </geometry>
+      </visual>
     </link>
     <link name="${arm_prefix}d405_color_frame">
@@ -33,29 +133,5 @@
     <link name="${arm_prefix}d405_infra2_optical_frame">
     </link>
-    <link name="${arm_prefix}robotiq_85_base_adapter_link">
-    </link>
-    <link name="${arm_prefix}robotiq_85_base_link">
-    </link>
-    <link name="${arm_prefix}robotiq_85_left_finger_link">
-    </link>
-    <link name="${arm_prefix}robotiq_85_left_finger_tip_link">
-    </link>
-    <link name="${arm_prefix}robotiq_85_left_inner_knuckle_link">
-    </link>
-    <link name="${arm_prefix}robotiq_85_left_knuckle_link">
-    </link>
-    <link name="${arm_prefix}robotiq_85_right_finger_link">
-    </link>
-    <link name="${arm_prefix}robotiq_85_right_finger_tip_link">
-    </link>
-    <link name="${arm_prefix}robotiq_85_right_inner_knuckle_link">
-    </link>
-    <link name="${arm_prefix}robotiq_85_right_knuckle_link">
-    </link>
     <link name="${arm_prefix}tcp">
-    </link>
-    <link name="${arm_prefix}fr3v2_ur_to_robotiq_link">
-    </link>
-    <link name="${arm_prefix}wrist_cam_mount_link">
     </link>
     <!-- ── Joints ────────────────────────────────────────── -->

Commit message: Add ALOHA fingertip variant and thread fingertip_style through macro chain
- Add robotiq_85_left/right_finger_tip_link_aloha.stl meshes (Adapted
  Fingertips - ALOHA Fingertip) to end effector mesh directory
- Add fingertip_style param (standard|aloha) to robotiq_2f85_d405_kinematics
  macro; ALOHA variant uses corrected rpy="1.5707963 0 -1.5707963" visual origin
- Thread fingertip_style through full macro chain: robotiq_2f85_d405 →
  franka_robot → fr3_duo → mobile_fr3_duo_v0_2 → top-level urdf.xacro arg
- Add --fingertip-style CLI flag to create_urdf.py; non-standard styles get
  a suffix in the output filename (e.g. mobile_fr3_duo_v0_2_robotiq_2f85_d405_aloha.urdf)

Co-Authored-By: Claude Sonnet 4.6 <noreply@anthropic.com>

File: end_effectors/robotiq_2f85_d405/robotiq_2f85_d405.urdf.xacro (robot description, xacro)
@@ -27,5 +27,6 @@
             xyz_ee:='0 0 0'
             rpy_ee:='0 0 -0.7853982'
-            description_pkg:='franka_description'">
+            description_pkg:='franka_description'
+            fingertip_style:='standard'">
     <!--
       Attachment joint: arm flange (link8) → fr3v2_ur_to_robotiq_link.
@@ -39,5 +40,5 @@
     </joint>
     <!-- All gripper + camera links and joints (prefixed for dual-arm safety) -->
-    <xacro:robotiq_2f85_d405_kinematics arm_prefix="${arm_prefix}" description_pkg="${description_pkg}"/>
+    <xacro:robotiq_2f85_d405_kinematics arm_prefix="${arm_prefix}" description_pkg="${description_pkg}" fingertip_style="${fingertip_style}"/>
   </xacro:macro>
 </robot>

File: end_effectors/robotiq_2f85_d405/robotiq_2f85_d405_kinematics.urdf.xacro (robot description, xacro)
@@ -15,5 +15,6 @@
   <xacro:macro name="robotiq_2f85_d405_kinematics"
                params="arm_prefix:=''
-                       description_pkg:='franka_description'">
+                       description_pkg:='franka_description'
+                       fingertip_style:='standard'">
     <!-- ── Links ─────────────────────────────────────────── -->
     <link name="${arm_prefix}fr3v2_ur_to_robotiq_link">
@@ -85,16 +86,32 @@
     <link name="${arm_prefix}robotiq_85_left_finger_tip_link">
       <visual>
-        <origin xyz="0 0 0" rpy="0 0 0"/>
-        <geometry>
-          <mesh filename="package://${description_pkg}/meshes/end_effectors/robotiq_2f85_d405/robotiq_85_left_finger_tip_link.stl"/>
-        </geometry>
+        <xacro:if value="${fingertip_style == 'aloha'}">
+          <origin xyz="0 0 0" rpy="1.5707963 0 -1.5707963"/>
+          <geometry>
+            <mesh filename="package://${description_pkg}/meshes/end_effectors/robotiq_2f85_d405/robotiq_85_left_finger_tip_link_aloha.stl"/>
+          </geometry>
+        </xacro:if>
+        <xacro:unless value="${fingertip_style == 'aloha'}">
+          <origin xyz="0 0 0" rpy="0 0 0"/>
+          <geometry>
+            <mesh filename="package://${description_pkg}/meshes/end_effectors/robotiq_2f85_d405/robotiq_85_left_finger_tip_link.stl"/>
+          </geometry>
+        </xacro:unless>
       </visual>
     </link>
     <link name="${arm_prefix}robotiq_85_right_finger_tip_link">
       <visual>
-        <origin xyz="0 0 0" rpy="0 0 0"/>
-        <geometry>
-          <mesh filename="package://${description_pkg}/meshes/end_effectors/robotiq_2f85_d405/robotiq_85_right_finger_tip_link.stl"/>
-        </geometry>
+        <xacro:if value="${fingertip_style == 'aloha'}">
+          <origin xyz="0 0 0" rpy="1.5707963 0 -1.5707963"/>
+          <geometry>
+            <mesh filename="package://${description_pkg}/meshes/end_effectors/robotiq_2f85_d405/robotiq_85_right_finger_tip_link_aloha.stl"/>
+          </geometry>
+        </xacro:if>
+        <xacro:unless value="${fingertip_style == 'aloha'}">
+          <origin xyz="0 0 0" rpy="0 0 0"/>
+          <geometry>
+            <mesh filename="package://${description_pkg}/meshes/end_effectors/robotiq_2f85_d405/robotiq_85_right_finger_tip_link.stl"/>
+          </geometry>
+        </xacro:unless>
       </visual>
     </link>

File: robots/common/franka_robot.xacro (robot description, xacro)
@@ -24,4 +24,5 @@
                       arm_prefix:=''
                       description_pkg:='franka_description'
+                      fingertip_style:='standard'
                       connected_to:='base'
                       is_async:=false
@@ -80,4 +81,5 @@
         rpy_ee="${rpy_ee}"
         description_pkg="${description_pkg}"
+        fingertip_style="${fingertip_style}"
       />
     </xacro:if>

File: robots/fr3_duo/fr3_duo.xacro (robot description, xacro)
@@ -31,5 +31,6 @@
             is_async:=false
             thread_priority:=50
-            is_mobile_fr3_duo:=false">
+            is_mobile_fr3_duo:=false
+            fingertip_style:='standard'">
     <xacro:property name="robot_types_list" value="${robot_types}"/>
     <xacro:property name="robot_ips_list" value="${robot_ips}"/>
@@ -81,4 +82,5 @@
           arm_prefix="${modified_prefix}"
           description_pkg="${description_pkg}"
+          fingertip_style="${fingertip_style}"
           connected_to="${arm_prefixes_list[i]}_base"
           is_async="${is_async}"

File: robots/mobile_fr3_duo_v0_2/mobile_fr3_duo_v0_2.urdf.xacro (robot description, xacro)
@@ -51,4 +51,6 @@
   <!-- Should the arms be used? -->
   <xacro:arg name="use_arms" default="true"/>
+  <!-- Fingertip style for robotiq_2f85_d405: 'standard' or 'aloha' -->
+  <xacro:arg name="fingertip_style" default="standard"/>
   <xacro:mobile_fr3_duo_v0_2
     robot_types="$(arg robot_types)"
@@ -65,4 +67,5 @@
     use_arms="$(arg use_arms)"
     no_prefix="$(arg no_prefix)"
+    fingertip_style="$(arg fingertip_style)"
     ee_id="$(arg ee_id)"
     special_connection="$(arg special_connection)"

File: robots/mobile_fr3_duo_v0_2/mobile_fr3_duo_v0_2.xacro (robot description, xacro)
@@ -25,5 +25,6 @@
             with_sc
             is_async:=false
-            thread_priority:=50">
+            thread_priority:=50
+            fingertip_style:='standard'">
     <xacro:include filename="$(find franka_description)/accessories/franka_spine_v0_1/franka_spine.xacro"/>
     <xacro:include filename="$(find franka_description)/robots/common/franka_robot.xacro"/>
@@ -91,4 +92,5 @@
       is_async="${is_async}"
       thread_priority="${thread_priority}"
+      fingertip_style="${fingertip_style}"
       is_mobile_fr3_duo="true"/>
     <xacro:if value="${gazebo}">
